File: phonopreamp/phonopreamp.kicad_pcb (KiCad board)
At the start: 2 copper layers, 91 x 58 mm, 99 parts, among them J1 16VAC, SW1 MFS201N-16-Z, U1 LM317LD, U2 LM337LMX, U3 LM4562, U4 LM4562

Commit message: Release revision B
Parts:
- U1: value LM317LD -> LM317LMX
Connections:
- J1 pad MP: (no net) -> GND
Routing:
- net GND: track 101.1 -> 108.7 mm
Other:
- board text added: "16VAC 500mA"
- board text added: "Phono preamp PA1-P06 rev B moving magnet type only"
- board text removed: "12VAC 500mA"
- board text removed: "Phono preamp and equalizer moving magnet type only"
